File: pcb/glowie/glowie.kicad_pcb (KiCad board)
At the start: 2 copper layers, 35 x 32.2 mm, 77 parts, among them J1 Conn_01x05_Pin, J2 Conn_01x04_Pin, J3 Battery, J4 Conn_01x01, Q1 SI2365EDS-T1-BE3, Q2 MMBT3906WT1G, Q3 NX7002BKWX, U1 LSM6DSV32XTR, U2 ESP32-C3-MINI-1, U3 DIO5508XS8, U4 NCP189CMTW330TAG, U5 74LVC2T45DC, U7 MIC2876-AYMT-TR

Commit message: mainboard new PCBA revision
- fix findings
Parts:
- C17: value 0.1uF -> 1uF
- R1, R2: value 33 -> 0
- R16: value 1M -> 100k
- R19: value 800k 1% -> 820k 1%
- R20: value 200k 1% -> 240k 1%
- R23: value 100k -> 10k
- R25: value 510k -> 1M
- R9: value 0.1 1% -> 0
Changed lines of the file:
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@@
 		)
 	)
-	(variants
-		(variant
-			(name "BQ297")
-		)
-	)
 	(footprint "Connector_Wire:SolderWire-0.5sqmm_1x01_D0.9mm_OD2.1mm"
 		(layer "F.Cu")
@@
 			)
 		)
-		(property "Value" "0.1 1%"
+		(property "Value" "0"
 			(at 0 1.17 180)
 			(unlocked yes)
@@
 			)
 		)
+		(property "Sim.Library" "/home/isaac/devel/glowie/pcb/pcb/Lib/sim/DLLFSD01LP3.spice.txt"
+			(at 0 0 0)
+			(unlocked yes)
+			(layer "F.Fab")
+			(hide yes)
+			(effects
+				(font
+					(size 1 1)
+					(thickness 0.15)
+				)
+			)
+		)
+		(property "Sim.Name" "DLLFSD01LP3"
+			(at 0 0 0)
+			(unlocked yes)
+			(layer "F.Fab")
+			(hide yes)
+			(effects
+				(font
+					(size 1 1)
+					(thickness 0.15)
+				)
+			)
+		)
 		(property ki_fp_filters "TO-???* *_Diode_* *SingleDiode* D_*")
 		(sheetname "/GP_Button/")
@@
 			)
 		)
+		(property "Sim.Library" "/home/isaac/devel/glowie/pcb/pcb/Lib/sim/DLLFSD01LP3.spice.txt"
+			(at 0 0 0)
+			(unlocked yes)
+			(layer "F.Fab")
+			(hide yes)
+			(effects
+				(font
+					(size 1 1)
+					(thickness 0.15)
+				)
+			)
+		)
+		(property "Sim.Name" "DLLFSD01LP3"
+			(at 0 0 0)
+			(unlocked yes)
+			(layer "F.Fab")
+			(hide yes)
+			(effects
+				(font
+					(size 1 1)
+					(thickness 0.15)
+				)
+			)
+		)
 		(property ki_fp_filters "TO-???* *_Diode_* *SingleDiode* D_*")
 		(sheetname "/GP_Button/")
@@
 			)
 		)
+		(property "Sim.Library" "/home/isaac/devel/glowie/pcb/pcb/Lib/sim/DLLFSD01LP3.spice.txt"
+			(at 0 0 0)
+			(unlocked yes)
+			(layer "F.Fab")
+			(hide yes)
+			(effects
+				(font
+					(size 1 1)
+					(thickness 0.15)
+				)
+			)
+		)
+		(property "Sim.Name" "DLLFSD01LP3"
+			(at 0 0 0)
+			(unlocked yes)
+			(layer "F.Fab")
+			(hide yes)
+			(effects
+				(font
+					(size 1 1)
+					(thickness 0.15)
+				)
+			)
+		)
 		(property ki_fp_filters "TO-???* *_Diode_* *SingleDiode* D_*")
 		(sheetname "/GP_Button/")
@@
 			)
 		)
-		(property "Value" "100k"
+		(property "Value" "10k"
 			(at 0 1.17 180)
 			(unlocked yes)
@@
 			)
 		)
-		(property "Value" "33"
+		(property "Value" "0"
 			(at 0 1.17 180)
 			(unlocked yes)
@@
 			)
 		)
-		(property "Value" "1M"
+		(property "Value" "100k"
 			(at 0 1.17 270)
 			(unlocked yes)
@@
 			)
 		)
+		(property "Sim.Library" "/home/isaac/devel/glowie/pcb/pcb/Lib/sim/DLLFSD01LP3.spice.txt"
+			(at 0 0 180)
+			(unlocked yes)
+			(layer "F.Fab")
+			(hide yes)
+			(effects
+				(font
+					(size 1 1)
+					(thickness 0.15)
+				)
+			)
+		)
+		(property "Sim.Name" "DLLFSD01LP3"
+			(at 0 0 180)
+			(unlocked yes)
+			(layer "F.Fab")
+			(hide yes)
+			(effects
+				(font
+					(size 1 1)
+					(thickness 0.15)
+				)
+			)
+		)
 		(property ki_fp_filters "TO-???* *_Diode_* *SingleDiode* D_*")
 		(sheetname "/GP_Button/")
@@
 		(sheetname "/Power/LED_converter/")
 		(sheetfile "led_converter.kicad_sch")
+		(units
+			(unit
+				(name "A")
+				(pins "1" "2")
+			)
+		)
 		(attr smd)
 		(duplicate_pad_numbers_are_jumpers no)
@@
 			)
 		)
+		(property "Sim.Library" "/home/isaac/devel/glowie/pcb/pcb/Lib/sim/DLLFSD01LP3.spice.txt"
+			(at 0 0 0)
+			(unlocked yes)
+			(layer "F.Fab")
+			(hide yes)
+			(effects
+				(font
+					(size 1 1)
+					(thickness 0.15)
+				)
+			)
+		)
+		(property "Sim.Name" "DLLFSD01LP3"
+			(at 0 0 0)
+			(unlocked yes)
+			(layer "F.Fab")
+			(hide yes)
+			(effects
+				(font
+					(size 1 1)
+					(thickness 0.15)
+				)
+			)
+		)
 		(property ki_fp_filters "TO-???* *_Diode_* *SingleDiode* D_*")
 		(sheetname "/GP_Button/")
@@
 			)
 		)
-		(property "Value" "800k 1%"
+		(property "Value" "820k 1%"
 			(at 0 1.17 270)
 			(unlocked yes)
@@
 			)
 		)
-		(property "Value" "0.1uF"
+		(property "Value" "1uF"
 			(at 0 1.16 180)
 			(unlocked yes)
@@
 			)
 		)
-		(attr smd)
+		(attr smd dnp)
 		(duplicate_pad_numbers_are_jumpers no)
 		(fp_line
@@
 			)
 		)
-		(property "Value" "200k 1%"
+		(property "Value" "240k 1%"
 			(at 0 1.17 270)
 			(unlocked yes)
@@
 			)
 		)
-		(property "Value" "510k"
+		(property "Value" "1M"
 			(at 0 1.17 180)
 			(unlocked yes)
@@
 			)
 		)
-		(property "Value" "33"
+		(property "Value" "0"
 			(at 0 1.17 180)
 			(unlocked yes)
