File: pcb/glowie/glowie.kicad_sch (KiCad schematic)
At the start: 34 parts, among them J1 Conn_01x05_Pin, J2 Conn_01x04_Pin, U1 LSM6DSV32XTR, U2 ESP32-C3-MINI-1, U5 74LVC2T45DC

Commit message: mainboard new PCBA revision
- fix findings
Parts:
- R1, R2: value 33 -> 0
- R9: value 0.1 1% -> 0
- U5: now not fitted
Changed lines of the file:
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@@
 			)
 		)
-		(property "Value" "0.1 1%"
+		(property "Value" "0"
 			(at 239.522 25.908 90)
 			(show_name no)
@@
 					(reference "R9")
 					(unit 1)
-					(variant
-						(name "BQ297")
-					)
 				)
 			)
@@
 					(reference "R11")
 					(unit 1)
-					(variant
-						(name "BQ297")
-					)
 				)
 			)
@@
 					(reference "C3")
 					(unit 1)
-					(variant
-						(name "BQ297")
-					)
 				)
 			)
@@
 		(on_board yes)
 		(in_pos_files yes)
-		(dnp no)
+		(dnp yes)
 		(property "Reference" "U5"
 			(at 213.7567 148.59 0)
@@
 					(reference "U2")
 					(unit 1)
-					(variant
-						(name "BQ297")
-					)
 				)
 			)
@@
 					(reference "C1")
 					(unit 1)
-					(variant
-						(name "BQ297")
-					)
 				)
 			)
@@
 			)
 		)
-		(property "Value" "33"
+		(property "Value" "0"
 			(at 69.85 48.26 90)
 			(show_name no)
@@
 					(reference "R2")
 					(unit 1)
-					(variant
-						(name "BQ297")
-					)
 				)
 			)
@@
 					(reference "R8")
 					(unit 1)
-					(variant
-						(name "BQ297")
-					)
 				)
 			)
@@
 					(reference "C4")
 					(unit 1)
-					(variant
-						(name "BQ297")
-					)
 				)
 			)
@@
 					(reference "U1")
 					(unit 1)
-					(variant
-						(name "BQ297")
-					)
 				)
 			)
@@
 					(reference "JP7")
 					(unit 1)
-					(variant
-						(name "BQ297")
-					)
 				)
 			)
@@
 					(reference "JP6")
 					(unit 1)
-					(variant
-						(name "BQ297")
-					)
 				)
 			)
@@
 			)
 		)
-		(property "Value" "33"
+		(property "Value" "0"
 			(at 69.85 35.814 90)
 			(show_name no)
@@
 					(reference "R1")
 					(unit 1)
-					(variant
-						(name "BQ297")
-					)
 				)
 			)
@@
 					(reference "C5")
 					(unit 1)
-					(variant
-						(name "BQ297")
-					)
 				)
 			)
@@
 					(reference "C7")
 					(unit 1)
-					(variant
-						(name "BQ297")
-					)
 				)
 			)
@@
 					(reference "C6")
 					(unit 1)
-					(variant
-						(name "BQ297")
-					)
 				)
 			)
@@
 					(reference "J1")
 					(unit 1)
-					(variant
-						(name "BQ297")
-						(dnp no)
-						(in_bom yes)
-					)
 				)
 			)
@@
 					(reference "J2")
 					(unit 1)
-					(variant
-						(name "BQ297")
-						(dnp no)
-						(in_bom yes)
-					)
 				)
 			)
@@
 					(reference "C2")
 					(unit 1)
-					(variant
-						(name "BQ297")
-					)
 				)
 			)
@@
 					(reference "R12")
 					(unit 1)
-					(variant
-						(name "BQ297")
-					)
 				)
 			)
