File: pcb/glowie/gp_button.kicad_sch (KiCad schematic)
At the start: 16 parts, among them Q2 MMBT3906WT1G, Q3 NX7002BKWX

Commit message: mainboard new PCBA revision
- fix findings
Parts:
- C17: value 0.1uF -> 1uF
- R23: value 100k -> 10k
- R25: value 510k -> 1M
Changed lines of the file:
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@@
 	)
 	(junction
-		(at 161.29 113.03)
-		(diameter 0)
-		(color 0 0 0 0)
-	)
-	(junction
 		(at 196.85 80.01)
 		(diameter 0)
@@
 	)
 	(junction
+		(at 161.29 113.03)
+		(diameter 0)
+		(color 0 0 0 0)
+	)
+	(junction
 		(at 167.64 86.36)
 		(diameter 0)
@@
 	(wire
 		(pts
-			(xy 194.31 113.03) (xy 209.55 113.03)
+			(xy 161.29 113.03) (xy 194.31 113.03)
 		)
 		(stroke
@@
 	(wire
 		(pts
-			(xy 196.85 80.01) (xy 196.85 83.82)
+			(xy 194.31 113.03) (xy 209.55 113.03)
 		)
 		(stroke
@@
 	(wire
 		(pts
-			(xy 139.7 86.36) (xy 139.7 97.79)
+			(xy 196.85 80.01) (xy 196.85 83.82)
 		)
 		(stroke
@@
 	(wire
 		(pts
-			(xy 109.22 77.47) (xy 118.11 77.47)
+			(xy 139.7 86.36) (xy 139.7 97.79)
 		)
 		(stroke
@@
 	(wire
 		(pts
-			(xy 139.7 105.41) (xy 139.7 113.03)
+			(xy 109.22 77.47) (xy 118.11 77.47)
 		)
 		(stroke
@@
 	(wire
 		(pts
-			(xy 114.3 46.99) (xy 109.22 46.99)
+			(xy 139.7 105.41) (xy 139.7 113.03)
 		)
 		(stroke
@@
 	(wire
 		(pts
-			(xy 161.29 113.03) (xy 194.31 113.03)
+			(xy 114.3 46.99) (xy 109.22 46.99)
 		)
 		(stroke
@@
 	(wire
 		(pts
+			(xy 161.29 113.03) (xy 161.29 119.38)
+		)
+		(stroke
+			(width 0)
+			(type default)
+		)
+	)
+	(wire
+		(pts
 			(xy 139.7 113.03) (xy 147.32 113.03)
 		)
@@
 	(wire
 		(pts
-			(xy 161.29 113.03) (xy 161.29 119.38)
-		)
-		(stroke
-			(width 0)
-			(type default)
-		)
-	)
-	(wire
-		(pts
 			(xy 92.71 77.47) (xy 109.22 77.47)
 		)
@@
 			)
 		)
+		(property "Sim.Library" "/home/isaac/devel/glowie/pcb/pcb/Lib/sim/DLLFSD01LP3.spice.txt"
+			(at 182.88 60.96 90)
+			(hide yes)
+			(show_name no)
+			(do_not_autoplace no)
+			(effects
+				(font
+					(size 1.27 1.27)
+				)
+			)
+		)
+		(property "Sim.Name" "DLLFSD01LP3"
+			(at 182.88 60.96 90)
+			(hide yes)
+			(show_name no)
+			(do_not_autoplace no)
+			(effects
+				(font
+					(size 1.27 1.27)
+				)
+			)
+		)
 		(pin "2"
 		)
@@
 			)
 		)
-		(property "Value" "100k"
+		(property "Value" "10k"
 			(at 151.13 109.22 90)
 			(show_name no)
@@
 			)
 		)
+		(property "Sim.Library" "/home/isaac/devel/glowie/pcb/pcb/Lib/sim/DLLFSD01LP3.spice.txt"
+			(at 110.49 102.87 0)
+			(hide yes)
+			(show_name no)
+			(do_not_autoplace no)
+			(effects
+				(font
+					(size 1.27 1.27)
+				)
+			)
+		)
+		(property "Sim.Name" "DLLFSD01LP3"
+			(at 110.49 102.87 0)
+			(hide yes)
+			(show_name no)
+			(do_not_autoplace no)
+			(effects
+				(font
+					(size 1.27 1.27)
+				)
+			)
+		)
 		(pin "2"
 		)
@@
 			)
 		)
+		(property "Sim.Library" "/home/isaac/devel/glowie/pcb/pcb/Lib/sim/DLLFSD01LP3.spice.txt"
+			(at 124.46 102.87 90)
+			(hide yes)
+			(show_name no)
+			(do_not_autoplace no)
+			(effects
+				(font
+					(size 1.27 1.27)
+				)
+			)
+		)
+		(property "Sim.Name" "DLLFSD01LP3"
+			(at 124.46 102.87 90)
+			(hide yes)
+			(show_name no)
+			(do_not_autoplace no)
+			(effects
+				(font
+					(size 1.27 1.27)
+				)
+			)
+		)
 		(pin "2"
 		)
@@
 			)
 		)
-		(property "Value" "0.1uF"
+		(property "Value" "1uF"
 			(at 165.1 124.4599 0)
 			(show_name no)
@@
 			)
 		)
-		(property "Value" "510k"
+		(property "Value" "1M"
 			(at 182.88 74.422 90)
 			(show_name no)
@@
 			)
 		)
+		(property "Sim.Library" "/home/isaac/devel/glowie/pcb/pcb/Lib/sim/DLLFSD01LP3.spice.txt"
+			(at 139.7 101.6 90)
+			(hide yes)
+			(show_name no)
+			(do_not_autoplace no)
+			(effects
+				(font
+					(size 1.27 1.27)
+				)
+			)
+		)
+		(property "Sim.Name" "DLLFSD01LP3"
+			(at 139.7 101.6 90)
+			(hide yes)
+			(show_name no)
+			(do_not_autoplace no)
+			(effects
+				(font
+					(size 1.27 1.27)
+				)
+			)
+		)
 		(pin "2"
 		)
@@
 			(at 109.22 62.23 90)
 			(hide yes)
+			(show_name no)
+			(do_not_autoplace no)
+			(effects
+				(font
+					(size 1.27 1.27)
+				)
+			)
+		)
+		(property "Sim.Library" "/home/isaac/devel/glowie/pcb/pcb/Lib/sim/DLLFSD01LP3.spice.txt"
+			(at 109.22 62.23 90)
+			(hide yes)
+			(show_name no)
+			(do_not_autoplace no)
+			(effects
+				(font
+					(size 1.27 1.27)
+				)
+			)
+		)
+		(property "Sim.Name" "DLLFSD01LP3"
+			(at 109.22 62.23 90)
+			(hide yes)
