File: pcb/glowie/gp_button_sim.kicad_sch (KiCad schematic)
At the start: 8 parts

Commit message: mainboard new PCBA revision
- fix findings
Parts:
- added R29: 10k, Resistor_SMD:R_0402_1005Metric, symbol Device:R
- V3: value 3.3 -> 3
- V4: value 3.7 -> 4.2
Connections:
- net GND: now also R29.1
- net GP_Button/LATCH: now also R29.2
- net VBUS_5V: no longer V2.1
- net VCC_3V3: no longer R28.2
Changed lines of the file:
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@@
-	)
-	(junction
-		(at 208.28 48.26)
-		(diameter 0)
-		(color 0 0 0 0)
 	)
 	(junction
@@
 		(color 0 0 0 0)
 	)
+	(junction
+		(at 105.41 105.41)
+		(diameter 0)
+		(color 0 0 0 0)
+	)
 	(wire
 		(pts
@@
 	(wire
 		(pts
+			(xy 105.41 119.38) (xy 105.41 123.19)
+		)
+		(stroke
+			(width 0)
+			(type default)
+		)
+	)
+	(wire
+		(pts
 			(xy 62.23 97.79) (xy 62.23 87.63)
 		)
@@
 	(wire
 		(pts
-			(xy 90.17 105.41) (xy 110.49 105.41)
+			(xy 90.17 105.41) (xy 105.41 105.41)
 		)
 		(stroke
@@
 	(wire
 		(pts
+			(xy 105.41 105.41) (xy 110.49 105.41)
+		)
+		(stroke
+			(width 0)
+			(type default)
+		)
+	)
+	(wire
+		(pts
 			(xy 54.61 82.55) (xy 54.61 87.63)
 		)
@@
 	(wire
 		(pts
-			(xy 90.17 91.44) (xy 90.17 93.98)
-		)
-		(stroke
-			(width 0)
-			(type default)
-		)
-	)
-	(wire
-		(pts
 			(xy 196.85 55.88) (xy 196.85 48.26)
 		)
@@
 	(wire
 		(pts
-			(xy 208.28 48.26) (xy 208.28 54.61)
-		)
-		(stroke
-			(width 0)
-			(type default)
-		)
-	)
-	(wire
-		(pts
 			(xy 196.85 48.26) (xy 208.28 48.26)
+		)
+		(stroke
+			(width 0)
+			(type default)
+		)
+	)
+	(wire
+		(pts
+			(xy 105.41 105.41) (xy 105.41 111.76)
 		)
 		(stroke
@@
 			)
 		)
-		(property "Value" "3.3"
+		(property "Value" "3"
 			(at 237.49 60.8301 0)
 			(show_name no)
@@
 			)
 		)
-		(property "Sim.Params" "y1=-1 y2=1 td=1 tr=2n tf=2n tw=0.02 per=5"
+		(property "Sim.Params" "y1=-1 y2=1 td=0 tr=2n tf=2n tw=30 per=60"
 			(at 67.1802 115.57 90)
 			(show_name no)
@@
 			)
 		)
-		(property "Value" "3.7"
+		(property "Value" "4.2"
 			(at 262.89 60.8301 0)
 			(show_name no)
@@
 				(path "/9c5b5a12-c6d6-47fd-bc0f-fd7712ded438"
 					(reference "V4")
+					(unit 1)
+				)
+			)
+		)
+	)
+	(symbol
+		(lib_id "Device:R")
+		(at 105.41 115.57 180)
+		(unit 1)
+		(body_style 1)
+		(exclude_from_sim no)
+		(in_bom no)
+		(on_board no)
+		(in_pos_files yes)
+		(dnp no)
+		(fields_autoplaced yes)
+		(property "Reference" "R29"
+			(at 107.95 114.2999 0)
+			(show_name no)
+			(do_not_autoplace no)
+			(effects
+				(font
+					(size 1.27 1.27)
+				)
+				(justify right)
+			)
+		)
+		(property "Value" "10k"
+			(at 107.95 116.8399 0)
+			(show_name no)
+			(do_not_autoplace no)
+			(effects
+				(font
+					(size 1.27 1.27)
+				)
+				(justify right)
+			)
+		)
+		(property "Footprint" "Resistor_SMD:R_0402_1005Metric"
+			(at 107.188 115.57 90)
+			(hide yes)
+			(show_name no)
+			(do_not_autoplace no)
+			(effects
+				(font
+					(size 1.27 1.27)
+				)
+			)
+		)
+		(property "Datasheet" ""
+			(at 105.41 115.57 0)
+			(hide yes)
+			(show_name no)
+			(do_not_autoplace no)
+			(effects
+				(font
+					(size 1.27 1.27)
+				)
+			)
+		)
+		(property "Description" "Resistor"
+			(at 105.41 115.57 0)
+			(hide yes)
+			(show_name no)
+			(do_not_autoplace no)
+			(effects
+				(font
+					(size 1.27 1.27)
+				)
+			)
+		)
+		(property "MPN" "0402 1M"
+			(at 105.41 115.57 0)
+			(hide yes)
+			(show_name no)
+			(do_not_autoplace no)
+			(effects
+				(font
+					(size 1.27 1.27)
+				)
+			)
+		)
+		(pin "1"
+		)
+		(pin "2"
+		)
+		(instances
+			(project "gp_button_sim"
+				(path "/0420817f-a395-4a26-909d-946f57998baf"
+					(reference "R655")
+					(unit 1)
+				)
+			)
+			(project "glowie"
+				(path "/9c5b5a12-c6d6-47fd-bc0f-fd7712ded438"
+					(reference "R29")
 					(unit 1)
 				)
@@
 					(unit 1)
 				)
+			)
+		)
+	)
+	(symbol
+		(lib_id "power:GND")
+		(at 105.41 123.19 0)
+		(unit 1)
+		(body_style 1)
+		(exclude_from_sim no)
+		(in_bom no)
+		(on_board no)
+		(in_pos_files no)
+		(dnp no)
+		(fields_autoplaced yes)
+		(property "Reference" "#PWR200"
+			(at 105.41 129.54 0)
+			(hide yes)
+			(show_name no)
+			(do_not_autoplace no)
+			(effects
+				(font
+					(size 1.27 1.27)
+				)
+			)
+		)
+		(property "Value" "GND"
+			(at 105.41 128.27 0)
+			(show_name no)
+			(do_not_autoplace no)
+			(effects
+				(font
+					(size 1.27 1.27)
+				)
+			)
+		)
+		(property "Footprint" ""
+			(at 105.41 123.19 0)
+			(hide yes)
+			(show_name no)
+			(do_not_autoplace no)
+			(effects
+				(font
+					(size 1.27 1.27)
+				)
+			)
+		)
+		(property "Datasheet" ""
+			(at 105.41 123.19 0)
+			(hide yes)
+			(show_name no)
+			(do_not_autoplace no)
+			(effects
+				(font
+					(size 1.27 1.27)
+				)
+			)
+		)
+		(property "Description" "Power symbol creates a global label with name \"GND\" , ground"
+			(at 105.41 123.19 0)
+			(hide yes)
+			(show_name no)
+			(do_not_autoplace no)
+			(effects
+				(font
+					(size 1.27 1.27)
+				)
+			)
+		)
+		(pin "1"
+		)
+		(instances
+			(project "gp_button_sim"
+				(path "/0420817f-a395-4a26-909d-946f57998baf"
+					(reference "#PWR01")
+					(unit 1)
+				)
+			)
+			(project "glowie"
+				(path "/9c5b5a12-c6d6-47fd-bc0f-fd7712ded438"
+					(reference "#PWR200")
+					(unit 1)
+				)
