File: pcb/glowie/led_converter.kicad_sch (KiCad schematic)
At the start: 7 parts, among them U7 MIC2876-AYMT-TR

Commit message: mainboard new PCBA revision
- fix findings
Parts:
- L1: footprint Inductor_SMD:L_Wuerth_PMCI-322510 -> glowie_footprints:Inductor_SRP3212
- R19: value 800k 1% -> 820k 1%
- R20: value 200k 1% -> 240k 1%
Changed lines of the file:
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@@
 			)
 		)
-		(property "Value" "800k 1%"
+		(property "Value" "820k 1%"
 			(at 173.99 91.4399 0)
 			(show_name no)
@@
 			)
 		)
-		(property "Value" "200k 1%"
+		(property "Value" "240k 1%"
 			(at 173.99 105.4099 0)
 			(show_name no)
@@
 					(reference "C16")
 					(unit 1)
-					(variant
-						(name "BQ297")
-					)
 				)
 			)
@@
 			)
 		)
-		(property "Footprint" "Inductor_SMD:L_Wuerth_PMCI-322510"
+		(property "Footprint" "glowie_footprints:Inductor_SRP3212"
 			(at 102.87 85.09 0)
 			(hide yes)
@@
 					(reference "L1")
 					(unit 1)
-					(variant
-						(name "BQ297")
-					)
 				)
 			)
@@
 					(reference "C15")
 					(unit 1)
-					(variant
-						(name "BQ297")
-					)
 				)
 			)
@@
 					(reference "U7")
 					(unit 1)
-					(variant
-						(name "BQ297")
-					)
 				)
 			)
@@
 					(reference "C14")
 					(unit 1)
-					(variant
-						(name "BQ297")
-					)
-				)
-			)
+				)
+			)
