File: pcb/glowie/power.kicad_sch (KiCad schematic)
At the start: 18 parts, among them J3 Battery, J4 Conn_01x01, Q1 SI2365EDS-T1-BE3, U3 DIO5508XS8, U4 NCP189CMTW330TAG

Commit message: mainboard new PCBA revision
- fix findings
Parts:
- R16: value 1M -> 100k
Changed lines of the file:
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@@
 					(reference "D1")
 					(unit 1)
-					(variant
-						(name "BQ297")
-					)
 				)
 			)
@@
 					(reference "C11")
 					(unit 1)
-					(variant
-						(name "BQ297")
-					)
 				)
 			)
@@
 					(reference "Q1")
 					(unit 1)
-					(variant
-						(name "BQ297")
-					)
 				)
 			)
@@
 					(reference "R15")
 					(unit 1)
-					(variant
-						(name "BQ297")
-					)
 				)
 			)
@@
 					(reference "F1")
 					(unit 1)
-					(variant
-						(name "BQ297")
-					)
 				)
 			)
@@
 					(reference "U3")
 					(unit 1)
-					(variant
-						(name "BQ297")
-					)
 				)
 			)
@@
 					(reference "U4")
 					(unit 1)
-					(variant
-						(name "BQ297")
-					)
 				)
 			)
@@
 					(reference "J3")
 					(unit 1)
-					(variant
-						(name "BQ297")
-					)
 				)
 			)
@@
 					(reference "C12")
 					(unit 1)
-					(variant
-						(name "BQ297")
-					)
 				)
 			)
@@
 					(reference "R14")
 					(unit 1)
-					(variant
-						(name "BQ297")
-					)
 				)
 			)
@@
 					(reference "C10")
 					(unit 1)
-					(variant
-						(name "BQ297")
-					)
 				)
 			)
@@
 			)
 		)
-		(property "Value" "1M"
+		(property "Value" "100k"
 			(at 130.8101 86.36 0)
 			(show_name no)
@@
 					(reference "R16")
 					(unit 1)
-					(variant
-						(name "BQ297")
-					)
 				)
 			)
@@
 					(reference "R13")
 					(unit 1)
-					(variant
-						(name "BQ297")
-					)
-				)
-			)
+				)
+			)
