File: pcb/panel/glowie_panel.kicad_pcb (KiCad board)
At the start: 2 copper layers, 12 x 12 mm, 10 parts, among them J1 Conn_01x04, J3 Conn_01x01, J4 Conn_01x01, J5 USB_C_Receptacle_USB2.0_16P, J6 Conn_01x01, SW1 SW_Push, U1 USBLC6-2SC6

Commit message: Fix panel routing
Parts:
- U1: footprint glowie_footprints:SOT-23-6L (USBLC6-2) -> Package_TO_SOT_SMD:SOT-23-6
- moved J1 0.13 mm to (175.5, 105.5)
Connections:
- J1 pad 1: /USB_D+ -> /USB_D-
- J1 pad 2: /USB_D- -> /USB_D+
- U1 pad 1: /USB_D- -> Net-(J5-D--PadA7)
- U1 pad 3: Net-(J5-D--PadA7) -> Net-(J5-D+-PadA6)
- U1 pad 4: Net-(J5-D+-PadA6) -> /USB_D+
- U1 pad 6: /USB_D+ -> /USB_D-
Routing:
- net GND: track 14.1 -> 0.00 mm, vias 1 -> 0
- net /USB_D+: track 1.75 -> 6.66 mm
- net Net-(J5-D--PadA7): track 7.14 -> 8.30 mm
- net /GPButton: track 7.98 -> 7.34 mm
- net Net-(J5-D+-PadA6): track 5.55 -> 6.10 mm
- net /USB_VBUS: vias 2 -> 4
Other:
- board text added: "V-"
- board text added: "v0rB"
- board text removed: "GND"
- board text removed: "V0.0"

Commit message: Panel routing improvements
Connections:
- J1 pad 1: /USB_D- -> /USB_D+
- J1 pad 2: /USB_D+ -> /USB_D-
- U1 pad 1: Net-(J5-D--PadA7) -> Net-(J5-D+-PadA6)
- U1 pad 3: Net-(J5-D+-PadA6) -> Net-(J5-D--PadA7)
- U1 pad 4: /USB_D+ -> /USB_D-
- U1 pad 6: /USB_D- -> /USB_D+
Routing:
- net /USB_D+: track 6.66 -> 3.24 mm
- net Net-(J5-D--PadA7): track 8.30 -> 5.16 mm
- net /USB_D-: track 3.30 -> 5.80 mm
- net Net-(J5-D+-PadA6): track 6.10 -> 7.48 mm
- net /USB_VBUS: vias 4 -> 2
