File: pcb/panel/glowie_panel.kicad_sch (KiCad schematic)
At the start: 10 parts, among them J1 Conn_01x04, J3 Conn_01x01, J4 Conn_01x01, J5 USB_C_Receptacle_USB2.0_16P, J6 Conn_01x01, SW1 SW_Push, U1 USBLC6-2SC6

Commit message: Fix panel routing
Parts:
- U1: footprint glowie_footprints:SOT-23-6L (USBLC6-2) -> Package_TO_SOT_SMD:SOT-23-6
Connections:
- net USB_D+: now also J1.2 (Pin_2), U1.4 (I/O2); no longer J1.1 (Pin_1), U1.6 (I/O1)
- net USB_D-: now also J1.1 (Pin_1), U1.6 (I/O1); no longer J1.2 (Pin_2), U1.1 (I/O1)
- net at J5.A7 (D-), J5.B7 (D-): now also U1.1 (I/O1); no longer U1.3 (I/O2)
- net at J5.A6 (D+), J5.B6 (D+): now also U1.3 (I/O2); no longer U1.4 (I/O2)
Other:
- moved on the sheet: J1, J3, J4, J6, SW1, U1

Commit message: Panel routing improvements
Connections:
- net USB_D+: now also J1.1 (Pin_1), U1.6 (I/O1); no longer J1.2 (Pin_2), U1.4 (I/O2)
- net USB_D-: now also J1.2 (Pin_2), U1.4 (I/O2); no longer J1.1 (Pin_1), U1.6 (I/O1)
- net at J5.A7 (D-), J5.B7 (D-): now also U1.3 (I/O2); no longer U1.1 (I/O1)
- net at J5.A6 (D+), J5.B6 (D+): now also U1.1 (I/O1); no longer U1.3 (I/O2)
Changed lines of the file:
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@@
 	(paper "A4")
 	(junction
+		(at 101.6 82.55)
+		(diameter 0)
+		(color 0 0 0 0)
+	)
+	(junction
 		(at 110.49 69.85)
 		(diameter 0)
@@
 	)
 	(junction
+		(at 81.28 102.87)
+		(diameter 0)
+		(color 0 0 0 0)
+	)
+	(junction
+		(at 123.19 102.87)
+		(diameter 0)
+		(color 0 0 0 0)
+	)
+	(junction
+		(at 132.08 62.23)
+		(diameter 0)
+		(color 0 0 0 0)
+	)
+	(junction
+		(at 110.49 102.87)
+		(diameter 0)
+		(color 0 0 0 0)
+	)
+	(junction
 		(at 101.6 77.47)
-		(diameter 0)
-		(color 0 0 0 0)
-	)
-	(junction
-		(at 101.6 82.55)
-		(diameter 0)
-		(color 0 0 0 0)
-	)
-	(junction
-		(at 81.28 102.87)
-		(diameter 0)
-		(color 0 0 0 0)
-	)
-	(junction
-		(at 123.19 102.87)
-		(diameter 0)
-		(color 0 0 0 0)
-	)
-	(junction
-		(at 132.08 62.23)
-		(diameter 0)
-		(color 0 0 0 0)
-	)
-	(junction
-		(at 110.49 102.87)
 		(diameter 0)
 		(color 0 0 0 0)
@@
 	(wire
 		(pts
+			(xy 120.65 82.55) (xy 123.19 85.09)
+		)
+		(stroke
+			(width 0)
+			(type default)
+		)
+	)
+	(wire
+		(pts
 			(xy 140.97 116.84) (xy 153.67 116.84)
 		)
@@
 	(wire
 		(pts
-			(xy 119.38 82.55) (xy 119.38 77.47)
+			(xy 116.84 82.55) (xy 116.84 77.47)
 		)
 		(stroke
@@
 	(wire
 		(pts
+			(xy 123.19 82.55) (xy 127 82.55)
+		)
+		(stroke
+			(width 0)
+			(type default)
+		)
+	)
+	(wire
+		(pts
 			(xy 110.49 102.87) (xy 123.19 102.87)
 		)
@@
 	(wire
 		(pts
+			(xy 120.65 85.09) (xy 114.3 85.09)
+		)
+		(stroke
+			(width 0)
+			(type default)
+		)
+	)
+	(wire
+		(pts
 			(xy 123.19 116.84) (xy 123.19 102.87)
 		)
@@
 	(wire
 		(pts
-			(xy 116.84 85.09) (xy 116.84 82.55)
+			(xy 114.3 85.09) (xy 114.3 82.55)
 		)
 		(stroke
@@
 	(wire
 		(pts
-			(xy 127 85.09) (xy 116.84 85.09)
-		)
-		(stroke
-			(width 0)
-			(type default)
-		)
-	)
-	(wire
-		(pts
-			(xy 127 82.55) (xy 119.38 82.55)
+			(xy 127 85.09) (xy 123.19 85.09)
+		)
+		(stroke
+			(width 0)
+			(type default)
+		)
+	)
+	(wire
+		(pts
+			(xy 116.84 82.55) (xy 120.65 82.55)
 		)
 		(stroke
@@
 	(wire
 		(pts
-			(xy 119.38 77.47) (xy 101.6 77.47)
+			(xy 120.65 85.09) (xy 123.19 82.55)
+		)
+		(stroke
+			(width 0)
+			(type default)
+		)
+	)
+	(wire
+		(pts
+			(xy 116.84 77.47) (xy 101.6 77.47)
 		)
 		(stroke
@@
 	(wire
 		(pts
-			(xy 116.84 82.55) (xy 101.6 82.55)
+			(xy 114.3 82.55) (xy 101.6 82.55)
 		)
 		(stroke
@@
 	)
 	(label "USB_D-"
-		(at 154.94 82.55 0)
+		(at 154.94 85.09 0)
 		(effects
 			(font
@@
 	)
 	(label "USB_D+"
-		(at 154.94 85.09 0)
+		(at 154.94 82.55 0)
 		(effects
 			(font
